File: PicoDebugInterface/PicoDebugInterface.kicad_pcb (KiCad board)
At the start: 2 copper layers, 6 parts, among them J1 Conn_02x05_Odd_Even, J2 SWDConnections, J3 I2C0_con, J4 I2C1_conn, J5 Conn_01x03_Female, U1 Pico

Commit message: almost done the board layout
Parts:
- moved J1 1.00 mm to (128.7, 62.0)
- moved J2 0.52 mm to (128.8, 66.5)
- moved J5 0.26 mm to (128.8, 55.8)
Connections:
- J1 pad 3: Earth -> GND
- J2 pad 2: Earth -> GND
Routing:
- net GND: track 0.00 -> 18.8 mm
- net /SWDIO: track 0.00 -> 18.8 mm, vias 0 -> 2
- net /SDA_0: track 0.00 -> 16.1 mm, vias 0 -> 2
- net /SWDCLK: track 0.00 -> 12.5 mm, vias 0 -> 2
- net /Uart_RX: track 0.00 -> 12.3 mm, vias 0 -> 2
- net /VBUS_OUT: track 0.00 -> 11.1 mm, vias 0 -> 2
- net /SDA_1: track 0.00 -> 8.94 mm
- net /SCL_1: track 0.00 -> 7.75 mm
- net /SCL_0: track 0.00 -> 7.11 mm
- net /SWO: track 0.00 -> 4.90 mm

Commit message: board sent out
Parts:
- J1: value Conn_02x05_Odd_Even -> Pico_D_V0.1
Other:
- board outline added: 15.1 x 11.8 mm
- board text added: "GND SCL_0 SDA_0"
- board text added: "SDA_0 SCL_0 GND"
- board text added: "SWO U_Rx V_Out"
- board text added: "SW_C GND SW_D"
Changed lines of the file:
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@@
       (outputformat 1)
       (mirror false)
-      (drillshape 1)
+      (drillshape 0)
       (scaleselection 1)
-      (outputdirectory "")
+      (outputdirectory "gerber/")
     )
   )
@@
       (effects (font (size 1 1) (thickness 0.15)))
     )
-    (fp_text value "SWDConnections" (at 1.27 -3.81 unlocked) (layer "F.Fab")
+    (fp_text value "SWDConnections" (at -13.5128 -0.9144 unlocked) (layer "F.Fab")
       (effects (font (size 1 1) (thickness 0.15)))
     )
@@
     (property "Sheetname" "")
     (attr through_hole)
-    (fp_text reference "J1" (at 5.588 4.318) (layer "F.SilkS")
-      (effects (font (size 1 1) (thickness 0.15)))
-    )
-    (fp_text value "Conn_02x05_Odd_Even" (at 1.143 -1.765) (layer "F.SilkS")
+    (fp_text reference "J1" (at -3.7338 2.1974) (layer "F.SilkS")
+      (effects (font (size 1 1) (thickness 0.15)))
+    )
+    (fp_text value "Pico_D_V0.1" (at 0.1778 -0.241 180) (layer "F.SilkS")
       (effects (font (size 1 1) (thickness 0.15)))
     )
@@
       (effects (font (size 1 1) (thickness 0.15)))
     )
-    (fp_text value "Conn_01x03_Female" (at 0 1.3335 unlocked) (layer "F.Fab")
+    (fp_text value "Conn_01x03_Female" (at -0.1016 -1.5113 unlocked) (layer "F.Fab")
       (effects (font (size 1 1) (thickness 0.15)))
     )
@@
       (net 52 "/SDA_0") (pinfunction "Pin_3") (pintype "passive"))
   )
-  (gr_rect (start 121.158 55.88) (end 136.398 67.7545) (layer "F.Cu") (width 0.2) (fill none))
+  (gr_rect (start 121.2088 55.9308) (end 136.3472 67.7164) (layer "Edge.Cuts") (width 0.1) (fill none))
+  (gr_text "SW_C  GND  SW_D\n" (at 128.8288 66.1924) (layer "F.SilkS")
+    (effects (font (size 0.5 0.5) (thickness 0.125)))
+  )
+  (gr_text "SWO U_Rx V_Out\n" (at 128.8796 57.5564) (layer "F.SilkS")
+    (effects (font (size 0.5 0.5) (thickness 0.125)))
+  )
+  (gr_text "GND SCL_0 SDA_0\n\n" (at 134.874 61.8744 90) (layer "F.SilkS")
+    (effects (font (size 0.5 0.5) (thickness 0.125)))
+  )
+  (gr_text "SDA_0 SCL_0 GND \n\n" (at 122.5804 61.8236 270) (layer "F.SilkS")
+    (effects (font (size 0.5 0.5) (thickness 0.125)))
+  )
   (segment (start 133.7945 67.1195) (end 133.858 67.056) (width 0.25) (layer "F.Cu") (net 1))
   (segment (start 131.318 67.1195) (end 133.7945 67.1195) (width 0.25) (layer "F.Cu") (net 1))
