File: PicoDebugInterface/PicoDebugInterface.kicad_sch (KiCad schematic)
At the start: 6 parts, among them J1 Conn_02x05_Odd_Even, J2 SWDConnections, J3 I2C0_con, J4 I2C1_conn, J5 Conn_01x03_Female, U1 Pico

Commit message: almost done the board layout
Connections:
- net Earth is gone; now on net GND: J1.3 (Pin_3), J2.2 (Pin_2)
Changed lines of the file:
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@@
     (pin "3")
-  )
-  (symbol (lib_id "power:Earth") (at 68.58 59.69 270) (unit 1)
-    (in_bom yes) (on_board yes) (fields_autoplaced)
-    (property "Reference" "#PWR01" (id 0) (at 62.23 59.69 0)
-      (effects (font (size 1.27 1.27)) hide)
-    )
-    (property "Value" "Earth" (id 1) (at 64.77 59.69 0)
-      (effects (font (size 1.27 1.27)) hide)
-    )
-    (property "Footprint" "" (id 2) (at 68.58 59.69 0)
-      (effects (font (size 1.27 1.27)) hide)
-    )
-    (property "Datasheet" "~" (id 3) (at 68.58 59.69 0)
-      (effects (font (size 1.27 1.27)) hide)
-    )
-    (pin "1")
   )
   (symbol (lib_id "Connector:Conn_01x03_Female") (at 190.5 74.93 180) (unit 1)
@@
     (pin "2")
     (pin "3")
+  )
+  (symbol (lib_id "power:GND") (at 167.64 107.95 0) (unit 1)
+    (in_bom yes) (on_board yes)
+    (property "Reference" "#PWR?" (id 0) (at 167.64 114.3 0)
+      (effects (font (size 1.27 1.27)) hide)
+    )
+    (property "Value" "GND" (id 1) (at 166.37 115.57 90)
+      (effects (font (size 1.27 1.27)) (justify left))
+    )
+    (property "Footprint" "" (id 2) (at 167.64 107.95 0)
+      (effects (font (size 1.27 1.27)) hide)
+    )
+    (property "Datasheet" "" (id 3) (at 167.64 107.95 0)
+      (effects (font (size 1.27 1.27)) hide)
+    )
+    (pin "1")
   )
   (symbol (lib_id "MCU_RaspberryPi_and_Boards:Pico") (at 166.37 58.42 0) (unit 1)
@@
     (pin "3")
   )
-  (symbol (lib_id "power:Earth") (at 167.64 107.95 0) (unit 1)
-    (in_bom yes) (on_board yes) (fields_autoplaced)
-    (property "Reference" "#PWR0101" (id 0) (at 167.64 114.3 0)
-      (effects (font (size 1.27 1.27)) hide)
-    )
-    (property "Value" "Earth" (id 1) (at 167.64 111.76 0)
-      (effects (font (size 1.27 1.27)) hide)
-    )
-    (property "Footprint" "" (id 2) (at 167.64 107.95 0)
-      (effects (font (size 1.27 1.27)) hide)
-    )
-    (property "Datasheet" "~" (id 3) (at 167.64 107.95 0)
-      (effects (font (size 1.27 1.27)) hide)
-    )
-    (pin "1")
-  )
   (symbol (lib_id "power:GND") (at 134.62 77.47 90) (unit 1)
     (in_bom yes) (on_board yes) (fields_autoplaced)
@@
     (pin "3")
   )
+  (symbol (lib_id "power:GND") (at 68.58 59.69 270) (unit 1)
+    (in_bom yes) (on_board yes)
+    (property "Reference" "#PWR0104" (id 0) (at 62.23 59.69 0)
+      (effects (font (size 1.27 1.27)) hide)
+    )
+    (property "Value" "GND" (id 1) (at 68.58 58.42 90)
+      (effects (font (size 1.27 1.27)) (justify left))
+    )
+    (property "Footprint" "" (id 2) (at 68.58 59.69 0)
+      (effects (font (size 1.27 1.27)) hide)
+    )
+    (property "Datasheet" "" (id 3) (at 68.58 59.69 0)
+      (effects (font (size 1.27 1.27)) hide)
+    )
+    (pin "1")
+  )
   (symbol (lib_id "power:GND") (at 195.58 77.47 90) (unit 1)
     (in_bom yes) (on_board yes) (fields_autoplaced)
@@
   )
   (symbol_instances
-    (path "/21d6bcf9-360f-480a-a98d-8ab260d764ed"
-      (reference "#PWR01") (unit 1) (value "Earth") (footprint "")
-    )
-    (path "/56a45817-28c2-4d40-9250-19fa3c830686"
-      (reference "#PWR0101") (unit 1) (value "Earth") (footprint "")
-    )
     (path "/fc741062-eba7-486a-9bdd-93694f3e20a0"
       (reference "#PWR0102") (unit 1) (value "GND") (footprint "")
@@
       (reference "#PWR0103") (unit 1) (value "GND") (footprint "")
     )
+    (path "/9da9d422-ea96-4b0e-9e08-0921956f20e7"
+      (reference "#PWR0104") (unit 1) (value "GND") (footprint "")
+    )
+    (path "/4b77e662-7c3a-4656-93f5-8b68eeba592d"
+      (reference "#PWR?") (unit 1) (value "GND") (footprint "")
+    )
     (path "/9b902966-ba16-4535-a541-f240bc694ecc"

Commit message: board sent out
Parts:
- J1: value Conn_02x05_Odd_Even -> DebugCon
Changed lines of the file:
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@@
   (symbol (lib_id "power:GND") (at 167.64 107.95 0) (unit 1)
     (in_bom yes) (on_board yes)
-    (property "Reference" "#PWR?" (id 0) (at 167.64 114.3 0)
+    (property "Reference" "#PWR0101" (id 0) (at 167.64 114.3 0)
       (effects (font (size 1.27 1.27)) hide)
     )
@@
     (in_bom yes) (on_board yes)
     (property "Reference" "J1" (id 0) (at 85.09 50.8 0))
-    (property "Value" "Conn_02x05_Odd_Even" (id 1) (at 85.09 53.34 0))
+    (property "Value" "DebugCon" (id 1) (at 85.09 53.34 0))
     (property "Footprint" "LocalFootprints:3220-10-0300-00-TR" (id 2) (at 83.82 62.23 0)
       (effects (font (size 1.27 1.27)) hide)
@@
   )
   (symbol_instances
+    (path "/4b77e662-7c3a-4656-93f5-8b68eeba592d"
+      (reference "#PWR0101") (unit 1) (value "GND") (footprint "")
+    )
     (path "/fc741062-eba7-486a-9bdd-93694f3e20a0"
       (reference "#PWR0102") (unit 1) (value "GND") (footprint "")
@@
       (reference "#PWR0104") (unit 1) (value "GND") (footprint "")
     )
-    (path "/4b77e662-7c3a-4656-93f5-8b68eeba592d"
-      (reference "#PWR?") (unit 1) (value "GND") (footprint "")
-    )
     (path "/9b902966-ba16-4535-a541-f240bc694ecc"
-      (reference "J1") (unit 1) (value "Conn_02x05_Odd_Even") (footprint "LocalFootprints:3220-10-0300-00-TR")
+      (reference "J1") (unit 1) (value "DebugCon") (footprint "LocalFootprints:3220-10-0300-00-TR")
     )
     (path "/02ffa30b-684c-4183-b5b2-dc4dccd1694f"

Commit message: pushed fix for the connector so it a staight through cable
Parts:
- U1: footprint MCU_RaspberryPi_and_Boards:RPi_Pico_SMD_TH -> RP-Pico Libraries:RPi_Pico_SMD_TH
Changed lines of the file:
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@@
     (property "Reference" "U1" (id 0) (at 166.37 26.67 0))
     (property "Value" "Pico" (id 1) (at 166.37 29.21 0))
-    (property "Footprint" "MCU_RaspberryPi_and_Boards:RPi_Pico_SMD_TH" (id 2) (at 166.37 58.42 90)
+    (property "Footprint" "RP-Pico Libraries:RPi_Pico_SMD_TH" (id 2) (at 166.37 58.42 90)
       (effects (font (size 1.27 1.27)) hide)
     )
@@
     )
     (path "/4fe21c75-0ccd-4490-98b1-8c922bb64cdc"
-      (reference "U1") (unit 1) (value "Pico") (footprint "MCU_RaspberryPi_and_Boards:RPi_Pico_SMD_TH")
+      (reference "U1") (unit 1) (value "Pico") (footprint "RP-Pico Libraries:RPi_Pico_SMD_TH")
     )
   )
