File: RaspberryPi_PicoProgrammer/RaspberryPi_PicoProgrammer.kicad_pcb (KiCad board)
At the start: 2 copper layers, 43.2 x 27.9 mm, 7 parts, among them J1 Conn_02x05_Odd_Even, J2 Conn_01x07_Male, J3 Conn_02x03_Odd_Even, J4 BM03B-SRSS-TBLFSN, U1 Pico

Commit message: added schematic for raspberry pi
Parts:
- removed U1: Pico, MCU_RaspberryPi_and_Boards:RPi_Pico_SMD_TH
- added J5: Raspberry_Pi_2_3, Connector_PinHeader_2.54mm:PinHeader_2x20_P2.54mm_Vertical, F.Cu at (150.8, 63.0)
- J2: value Conn_01x07_Male -> Conn_01x03_Male; footprint Connector_PinSocket_2.54mm:PinSocket_1x07_P2.54mm_Horizontal -> Connector_PinHeader_2.54mm:PinHeader_1x03_P2.54mm_Horizontal
- moved J2 45.1 mm to (146.1, 111.0), turned to 180 degrees
- moved JP1 17.7 mm to (138.9, 66.5), turned to 90 degrees
- moved JP2 17.1 mm to (138.9, 62.6), turned to 90 degrees
- moved J1 13.5 mm to (140.0, 84.2), turned to 90 degrees
- moved J3 10.4 mm to (137.6, 71.2), turned to 90 degrees
- moved J4 5.99 mm to (138.4, 96.2), turned to -90 degrees
Connections:
- J2 pad 1: /SCL_0 -> /SWDCLK
- J2 pad 2: /SWDCLK -> Earth
- J2 pad 3: Earth -> /SWO
Other:
- board size 43.2 x 27.9 mm -> 20.2 x 55.2 mm

Commit message: almost done the board layout
Parts:
- moved JP2 4.73 mm to (141.6, 66.5), turned to -90 degrees
- moved JP1 4.57 mm to (141.5, 62.7), turned to -90 degrees
- moved J1 0.62 mm to (139.7, 83.7), turned to -90 degrees
Connections:
- net Earth renamed GND
- J3 pad 2: /SW0 -> /SWO
Routing:
- net /SWO: track 0.00 -> 60.1 mm, vias 0 -> 2
- net /SDA_1: track 0.00 -> 37.8 mm, vias 0 -> 1
- net /SWDCLK: track 0.00 -> 35.6 mm
- net /SWDIO: track 0.00 -> 34.8 mm, vias 0 -> 2
- net /SDA_0: track 0.00 -> 32.4 mm, vias 0 -> 1
- net /power_output: track 0.00 -> 30.4 mm, vias 0 -> 1
- net /SCL_1: track 0.00 -> 30.2 mm, vias 0 -> 1
- net /SCL_0: track 0.00 -> 21.2 mm
- net /UartTX: track 0.00 -> 15.1 mm
- net Net-(J5-Pad2): track 0.00 -> 12.6 mm
- net Net-(J5-Pad1): track 0.00 -> 10.6 mm
Other:
- outline, holes or cut-outs redrawn

Commit message: board sent out
Parts:
- J1: value Conn_02x05_Odd_Even -> Pi_Pico_debuger_V0.1
- J3: value Conn_02x03_Odd_Even -> Conn_Extra
- J4: value BM03B-SRSS-TBLFSN -> JST_Pico
- renumbered JP2 to 3.3, JP1 to 5v, J2 to SWD_Headers
Connections:
- J5 pad 14: unconnected-(J5-Pad14) -> GND
- J5 pad 20: unconnected-(J5-Pad20) -> GND
- J5 pad 25: unconnected-(J5-Pad25) -> GND
- J5 pad 30: unconnected-(J5-Pad30) -> GND
- J5 pad 34: unconnected-(J5-Pad34) -> GND
- J5 pad 39: unconnected-(J5-Pad39) -> GND
- J5 pad 6: unconnected-(J5-Pad6) -> GND
- J5 pad 9: unconnected-(J5-Pad9) -> GND
Routing:
- net /SWDCLK: track 35.6 -> 53.4 mm, vias 0 -> 2
- net GND: track 0.00 -> 7.05 mm, vias 0 -> 2
- added copper zone on B.Cu, net GND
Other:
- board size 20.2 x 55.2 mm -> 20.9 x 55.1 mm
- board text added: "RX C0 C1"
- board text added: "TX D0 D1"
