File: RaspberryPi_PicoProgrammer/RaspberryPi_PicoProgrammer.kicad_sch (KiCad schematic)
At the start: 7 parts, among them J1 Conn_02x05_Odd_Even, J2 Conn_01x07_Male, J3 Conn_02x03_Odd_Even, J4 BM03B-SRSS-TBLFSN, U1 Pico

Commit message: added schematic for raspberry pi
Parts:
- removed J2: Conn_01x07_Male, Connector_PinSocket_2.54mm:PinSocket_1x07_P2.54mm_Horizontal, symbol Connector:Conn_01x07_Male
- removed U1: Pico, MCU_RaspberryPi_and_Boards:RPi_Pico_SMD_TH, symbol MCU_RaspberryPi_and_Boards:Pico
- added J2: Conn_01x03_Male, Connector_PinHeader_2.54mm:PinHeader_1x03_P2.54mm_Horizontal, symbol Connector:Conn_01x03_Male
- added J5: Raspberry_Pi_2_3, Connector_PinHeader_2.54mm:PinHeader_2x20_P2.54mm_Vertical, symbol Connector:Raspberry_Pi_2_3
Connections:
- net Earth: now also J2.2 (Pin_2)
- net SCL_0: now also J5.5 (SCL/GPIO3)
- net SCL_1: now also J5.28 (ID_SC/GPIO1)
- net SDA_0: now also J5.3 (SDA/GPIO2)
- net SDA_1: now also J5.27 (ID_SD/GPIO0)
- net SWDCLK: now also J2.1 (Pin_1), J5.22 (GPIO25)
- net SWDIO: now also J5.18 (GPIO24)
- net SWO: now also J2.3 (Pin_3), J5.10 (GPIO15/RXD)
- net UartTX: now also J5.8 (GPIO14/TXD)
- net at JP1.1 (A): now also J5.2 (5V)
- net at JP2.1 (A): now also J5.1 (3V3)
Other:
- moved on the sheet: J4, JP1, JP2

Commit message: almost done the board layout
Connections:
- net SW0 is gone; now on net SWO: J3.2 (Pin_2)
- net Earth renamed GND
Changed lines of the file:
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@@
     (effects (font (size 1.27 1.27)) (justify right bottom))
   )
-  (label "SW0" (at 130.81 101.6 0)
+  (label "SWO" (at 130.81 101.6 0)
     (effects (font (size 1.27 1.27)) (justify left bottom))
   )
@@
     (pin "9")
   )
-  (symbol (lib_id "power:Earth") (at 102.87 66.04 270) (unit 1)
-    (in_bom yes) (on_board yes) (fields_autoplaced)
-    (property "Reference" "#PWR01" (id 0) (at 96.52 66.04 0)
-      (effects (font (size 1.27 1.27)) hide)
-    )
-    (property "Value" "Earth" (id 1) (at 99.06 66.04 0)
-      (effects (font (size 1.27 1.27)) hide)
-    )
-    (property "Footprint" "" (id 2) (at 102.87 66.04 0)
-      (effects (font (size 1.27 1.27)) hide)
-    )
-    (property "Datasheet" "~" (id 3) (at 102.87 66.04 0)
+  (symbol (lib_id "power:GND") (at 127 36.83 90) (unit 1)
+    (in_bom yes) (on_board yes) (fields_autoplaced)
+    (property "Reference" "#PWR?" (id 0) (at 133.35 36.83 0)
+      (effects (font (size 1.27 1.27)) hide)
+    )
+    (property "Value" "GND" (id 1) (at 130.81 36.8299 90)
+      (effects (font (size 1.27 1.27)) (justify right))
+    )
+    (property "Footprint" "" (id 2) (at 127 36.83 0)
+      (effects (font (size 1.27 1.27)) hide)
+    )
+    (property "Datasheet" "" (id 3) (at 127 36.83 0)
       (effects (font (size 1.27 1.27)) hide)
     )
@@
     (pin "1")
     (pin "2")
-  )
-  (symbol (lib_id "power:Earth") (at 127 36.83 90) (unit 1)
-    (in_bom yes) (on_board yes) (fields_autoplaced)
-    (property "Reference" "#PWR0101" (id 0) (at 133.35 36.83 0)
-      (effects (font (size 1.27 1.27)) hide)
-    )
-    (property "Value" "Earth" (id 1) (at 130.81 36.83 0)
-      (effects (font (size 1.27 1.27)) hide)
-    )
-    (property "Footprint" "" (id 2) (at 127 36.83 0)
-      (effects (font (size 1.27 1.27)) hide)
-    )
-    (property "Datasheet" "~" (id 3) (at 127 36.83 0)
-      (effects (font (size 1.27 1.27)) hide)
-    )
-    (pin "1")
   )
   (symbol (lib_id "Connector:Conn_01x03_Male") (at 121.92 36.83 0) (unit 1)
@@
     (pin "2")
     (pin "3")
+  )
+  (symbol (lib_id "power:GND") (at 168.91 125.73 180) (unit 1)
+    (in_bom yes) (on_board yes) (fields_autoplaced)
+    (property "Reference" "#PWR0103" (id 0) (at 168.91 119.38 0)
+      (effects (font (size 1.27 1.27)) hide)
+    )
+    (property "Value" "GND" (id 1) (at 171.45 124.4599 0)
+      (effects (font (size 1.27 1.27)) (justify right))
+    )
+    (property "Footprint" "" (id 2) (at 168.91 125.73 0)
+      (effects (font (size 1.27 1.27)) hide)
+    )
+    (property "Datasheet" "" (id 3) (at 168.91 125.73 0)
+      (effects (font (size 1.27 1.27)) hide)
+    )
+    (pin "1")
   )
   (symbol (lib_id "Connector_Generic:Conn_02x05_Odd_Even") (at 118.11 68.58 0) (unit 1)
@@
     (pin "9")
   )
-  (symbol (lib_id "power:Earth") (at 168.91 125.73 180) (unit 1)
-    (in_bom yes) (on_board yes) (fields_autoplaced)
-    (property "Reference" "#PWR0102" (id 0) (at 168.91 119.38 0)
-      (effects (font (size 1.27 1.27)) hide)
-    )
-    (property "Value" "Earth" (id 1) (at 168.91 121.92 0)
-      (effects (font (size 1.27 1.27)) hide)
-    )
-    (property "Footprint" "" (id 2) (at 168.91 125.73 0)
-      (effects (font (size 1.27 1.27)) hide)
-    )
-    (property "Datasheet" "~" (id 3) (at 168.91 125.73 0)
-      (effects (font (size 1.27 1.27)) hide)
-    )
-    (pin "1")
-  )
   (symbol (lib_id "Connector_Generic:Conn_02x03_Odd_Even") (at 123.19 104.14 0) (unit 1)
     (in_bom yes) (on_board yes) (fields_autoplaced)
@@
     (pin "3")
   )
+  (symbol (lib_id "power:GND") (at 102.87 66.04 270) (unit 1)
+    (in_bom yes) (on_board yes) (fields_autoplaced)
+    (property "Reference" "#PWR0102" (id 0) (at 96.52 66.04 0)
+      (effects (font (size 1.27 1.27)) hide)
+    )
+    (property "Value" "GND" (id 1) (at 99.06 66.0399 90)
+      (effects (font (size 1.27 1.27)) (justify right))
+    )
+    (property "Footprint" "" (id 2) (at 102.87 66.04 0)
+      (effects (font (size 1.27 1.27)) hide)
+    )
+    (property "Datasheet" "" (id 3) (at 102.87 66.04 0)
+      (effects (font (size 1.27 1.27)) hide)
+    )
+    (pin "1")
+  )
   (sheet_instances
     (path "/" (page "1"))
   )
   (symbol_instances
-    (path "/21d6bcf9-360f-480a-a98d-8ab260d764ed"
-      (reference "#PWR01") (unit 1) (value "Earth") (footprint "")
-    )
-    (path "/6eaf7757-5114-4ceb-bc89-5da22eb3e84a"
-      (reference "#PWR0101") (unit 1) (value "Earth") (footprint "")
-    )
-    (path "/a0a28fa4-b96b-4a66-a268-94b1e9e96d9a"
-      (reference "#PWR0102") (unit 1) (value "Earth") (footprint "")
+    (path "/fe11ca85-fcab-4900-9be1-2bca707624fd"
+      (reference "#PWR0102") (unit 1) (value "GND") (footprint "")
+    )
+    (path "/911ed9c0-0645-4b6c-8777-5708aeacb3fb"
+      (reference "#PWR0103") (unit 1) (value "GND") (footprint "")
+    )
+    (path "/2dc3733a-9d58-4877-8e6e-e1d8cbfa0c4a"
+      (reference "#PWR?") (unit 1) (value "GND") (footprint "")
     )
     (path "/9b902966-ba16-4535-a541-f240bc694ecc"

Commit message: board sent out
Connections:
- net GND: now also J5.14 (GND), J5.20 (GND), J5.25 (GND), J5.30 (GND), J5.34 (GND), J5.39 (GND), J5.6 (GND), J5.9 (GND)
Changed lines of the file:
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@@
     (pin "2")
+  )
+  (symbol (lib_id "power:GND") (at 172.72 109.22 0) (unit 1)
+    (in_bom yes) (on_board yes) (fields_autoplaced)
+    (property "Reference" "#PWR?" (id 0) (at 172.72 115.57 0)
+      (effects (font (size 1.27 1.27)) hide)
+    )
+    (property "Value" "GND" (id 1) (at 175.26 110.4899 0)
+      (effects (font (size 1.27 1.27)) (justify left))
+    )
+    (property "Footprint" "" (id 2) (at 172.72 109.22 0)
+      (effects (font (size 1.27 1.27)) hide)
+    )
+    (property "Datasheet" "" (id 3) (at 172.72 109.22 0)
+      (effects (font (size 1.27 1.27)) hide)
+    )
+    (pin "1")
   )
   (symbol (lib_id "Connector:Raspberry_Pi_2_3") (at 175.26 76.2 0) (unit 1)
@@
     (pin "2")
   )
+  (symbol (lib_id "power:GND") (at 182.88 109.22 0) (unit 1)
+    (in_bom yes) (on_board yes) (fields_autoplaced)
+    (property "Reference" "#PWR?" (id 0) (at 182.88 115.57 0)
+      (effects (font (size 1.27 1.27)) hide)
+    )
+    (property "Value" "GND" (id 1) (at 185.42 110.4899 0)
+      (effects (font (size 1.27 1.27)) (justify left))
+    )
+    (property "Footprint" "" (id 2) (at 182.88 109.22 0)
+      (effects (font (size 1.27 1.27)) hide)
+    )
+    (property "Datasheet" "" (id 3) (at 182.88 109.22 0)
+      (effects (font (size 1.27 1.27)) hide)
+    )
+    (pin "1")
+  )
+  (symbol (lib_id "power:GND") (at 175.26 109.22 0) (unit 1)
+    (in_bom yes) (on_board yes) (fields_autoplaced)
+    (property "Reference" "#PWR?" (id 0) (at 175.26 115.57 0)
+      (effects (font (size 1.27 1.27)) hide)
+    )
+    (property "Value" "GND" (id 1) (at 177.8 110.4899 0)
+      (effects (font (size 1.27 1.27)) (justify left))
+    )
+    (property "Footprint" "" (id 2) (at 175.26 109.22 0)
+      (effects (font (size 1.27 1.27)) hide)
+    )
+    (property "Datasheet" "" (id 3) (at 175.26 109.22 0)
+      (effects (font (size 1.27 1.27)) hide)
+    )
+    (pin "1")
+  )
   (symbol (lib_id "Connector:Conn_01x03_Male") (at 121.92 36.83 0) (unit 1)
     (in_bom yes) (on_board yes) (fields_autoplaced)
@@
     (pin "9")
   )
+  (symbol (lib_id "power:GND") (at 167.64 109.22 0) (unit 1)
+    (in_bom yes) (on_board yes) (fields_autoplaced)
+    (property "Reference" "#PWR?" (id 0) (at 167.64 115.57 0)
+      (effects (font (size 1.27 1.27)) hide)
+    )
+    (property "Value" "GND" (id 1) (at 170.18 110.4899 0)
+      (effects (font (size 1.27 1.27)) (justify left))
+    )
+    (property "Footprint" "" (id 2) (at 167.64 109.22 0)
+      (effects (font (size 1.27 1.27)) hide)
+    )
+    (property "Datasheet" "" (id 3) (at 167.64 109.22 0)
+      (effects (font (size 1.27 1.27)) hide)
+    )
+    (pin "1")
+  )
+  (symbol (lib_id "power:GND") (at 165.1 109.22 0) (unit 1)
+    (in_bom yes) (on_board yes) (fields_autoplaced)
+    (property "Reference" "#PWR?" (id 0) (at 165.1 115.57 0)
+      (effects (font (size 1.27 1.27)) hide)
+    )
+    (property "Value" "GND" (id 1) (at 167.64 110.4899 0)
+      (effects (font (size 1.27 1.27)) (justify left))
+    )
+    (property "Footprint" "" (id 2) (at 165.1 109.22 0)
+      (effects (font (size 1.27 1.27)) hide)
+    )
+    (property "Datasheet" "" (id 3) (at 165.1 109.22 0)
+      (effects (font (size 1.27 1.27)) hide)
+    )
+    (pin "1")
+  )
+  (symbol (lib_id "power:GND") (at 177.8 109.22 0) (unit 1)
+    (in_bom yes) (on_board yes) (fields_autoplaced)
+    (property "Reference" "#PWR?" (id 0) (at 177.8 115.57 0)
+      (effects (font (size 1.27 1.27)) hide)
+    )
+    (property "Value" "GND" (id 1) (at 180.34 110.4899 0)
+      (effects (font (size 1.27 1.27)) (justify left))
+    )
+    (property "Footprint" "" (id 2) (at 177.8 109.22 0)
+      (effects (font (size 1.27 1.27)) hide)
+    )
+    (property "Datasheet" "" (id 3) (at 177.8 109.22 0)
+      (effects (font (size 1.27 1.27)) hide)
+    )
+    (pin "1")
+  )
+  (symbol (lib_id "power:GND") (at 180.34 109.22 0) (unit 1)
+    (in_bom yes) (on_board yes) (fields_autoplaced)
+    (property "Reference" "#PWR?" (id 0) (at 180.34 115.57 0)
+      (effects (font (size 1.27 1.27)) hide)
+    )
+    (property "Value" "GND" (id 1) (at 182.88 110.4899 0)
+      (effects (font (size 1.27 1.27)) (justify left))
+    )
+    (property "Footprint" "" (id 2) (at 180.34 109.22 0)
+      (effects (font (size 1.27 1.27)) hide)
+    )
+    (property "Datasheet" "" (id 3) (at 180.34 109.22 0)
+      (effects (font (size 1.27 1.27)) hide)
+    )
+    (pin "1")
+  )
   (symbol (lib_id "Connector_Generic:Conn_02x03_Odd_Even") (at 123.19 104.14 0) (unit 1)
     (in_bom yes) (on_board yes) (fields_autoplaced)
@@
     (pin "3")
   )
+  (symbol (lib_id "power:GND") (at 170.18 109.22 0) (unit 1)
+    (in_bom yes) (on_board yes) (fields_autoplaced)
+    (property "Reference" "#PWR?" (id 0) (at 170.18 115.57 0)
+      (effects (font (size 1.27 1.27)) hide)
+    )
+    (property "Value" "GND" (id 1) (at 172.72 110.4899 0)
+      (effects (font (size 1.27 1.27)) (justify left))
+    )
+    (property "Footprint" "" (id 2) (at 170.18 109.22 0)
+      (effects (font (size 1.27 1.27)) hide)
+    )
+    (property "Datasheet" "" (id 3) (at 170.18 109.22 0)
+      (effects (font (size 1.27 1.27)) hide)
+    )
+    (pin "1")
+  )
   (symbol (lib_id "power:GND") (at 102.87 66.04 270) (unit 1)
     (in_bom yes) (on_board yes) (fields_autoplaced)
@@
       (reference "#PWR0103") (unit 1) (value "GND") (footprint "")
     )
+    (path "/148c1fef-b661-460b-a57a-325322a15ece"
+      (reference "#PWR?") (unit 1) (value "GND") (footprint "")
+    )
     (path "/2dc3733a-9d58-4877-8e6e-e1d8cbfa0c4a"
       (reference "#PWR?") (unit 1) (value "GND") (footprint "")
     )
+    (path "/3146ca1f-eed7-4baa-9733-67c1d02e5784"
+      (reference "#PWR?") (unit 1) (value "GND") (footprint "")
+    )
+    (path "/60940c6c-27ab-4fda-8fce-85de9b7166e0"
+      (reference "#PWR?") (unit 1) (value "GND") (footprint "")
+    )
+    (path "/ab3158bc-e462-4ae6-93b7-eb9a1d8fd8be"
+      (reference "#PWR?") (unit 1) (value "GND") (footprint "")
+    )
+    (path "/af81e9b3-8f66-48b0-834e-d6d8bce921bf"
+      (reference "#PWR?") (unit 1) (value "GND") (footprint "")
+    )
+    (path "/b24511b1-2c84-43ba-8736-fb8e70ff6c1d"
+      (reference "#PWR?") (unit 1) (value "GND") (footprint "")
+    )
+    (path "/cd4f74bf-5bbd-453d-bf71-0d8a83165477"
+      (reference "#PWR?") (unit 1) (value "GND") (footprint "")
+    )
+    (path "/fddcbc36-8d82-4d5d-9795-3829c0452e89"
+      (reference "#PWR?") (unit 1) (value "GND") (footprint "")
+    )
