File: PicoProbeProgrammerBoard/PicoProbeProgrammerBoard.kicad_sch (KiCad schematic)
At the start: 7 parts, among them J1 Conn_02x05_Odd_Even, J2 Conn_01x07_Male, J3 Conn_02x03_Odd_Even, J4 BM03B-SRSS-TBLFSN, U1 Pico

Commit message: almost done the board layout
Connections:
- net Earth is gone; now on net GND: J1.3 (Pin_3), J2.3 (Pin_3), J4.2, U1.8 (GND)
- net SW0 is gone; now on net SWO: J3.2 (Pin_2)
- net GND: now reaches U1.13 (GND)
- net GND: now also U1.18 (GND), U1.23 (GND), U1.28 (GND)
Changed lines of the file:
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@@
-    (stroke (width 0) (type default) (color 0 0 0 0))
-  )
-  (wire (pts (xy 130.81 36.83) (xy 130.81 35.56))
     (stroke (width 0) (type default) (color 0 0 0 0))
   )
@@
     (effects (font (size 1.27 1.27)) (justify right bottom))
   )
-  (label "SW0" (at 130.81 101.6 0)
+  (label "SWO" (at 130.81 101.6 0)
     (effects (font (size 1.27 1.27)) (justify left bottom))
   )
@@
     (pin "2")
   )
-  (symbol (lib_id "power:Earth") (at 102.87 66.04 270) (unit 1)
-    (in_bom yes) (on_board yes) (fields_autoplaced)
-    (property "Reference" "#PWR01" (id 0) (at 96.52 66.04 0)
-      (effects (font (size 1.27 1.27)) hide)
-    )
-    (property "Value" "Earth" (id 1) (at 99.06 66.04 0)
-      (effects (font (size 1.27 1.27)) hide)
-    )
-    (property "Footprint" "" (id 2) (at 102.87 66.04 0)
-      (effects (font (size 1.27 1.27)) hide)
-    )
-    (property "Datasheet" "~" (id 3) (at 102.87 66.04 0)
+  (symbol (lib_id "power:GND") (at 166.37 102.87 180) (unit 1)
+    (in_bom yes) (on_board yes)
+    (property "Reference" "#PWR0103" (id 0) (at 166.37 96.52 0)
+      (effects (font (size 1.27 1.27)) hide)
+    )
+    (property "Value" "GND" (id 1) (at 166.3701 99.06 90)
+      (effects (font (size 1.27 1.27)) (justify right))
+    )
+    (property "Footprint" "" (id 2) (at 166.37 102.87 0)
+      (effects (font (size 1.27 1.27)) hide)
+    )
+    (property "Datasheet" "" (id 3) (at 166.37 102.87 0)
+      (effects (font (size 1.27 1.27)) hide)
+    )
+    (pin "1")
+  )
+  (symbol (lib_id "power:GND") (at 148.59 64.77 270) (unit 1)
+    (in_bom yes) (on_board yes)
+    (property "Reference" "#PWR0107" (id 0) (at 142.24 64.77 0)
+      (effects (font (size 1.27 1.27)) hide)
+    )
+    (property "Value" "GND" (id 1) (at 142.24 64.77 90)
+      (effects (font (size 1.27 1.27)) (justify left))
+    )
+    (property "Footprint" "" (id 2) (at 148.59 64.77 0)
+      (effects (font (size 1.27 1.27)) hide)
+    )
+    (property "Datasheet" "" (id 3) (at 148.59 64.77 0)
       (effects (font (size 1.27 1.27)) hide)
     )
@@
     (pin "2")
   )
-  (symbol (lib_id "power:Earth") (at 143.51 52.07 0) (unit 1)
-    (in_bom yes) (on_board yes) (fields_autoplaced)
-    (property "Reference" "#PWR02" (id 0) (at 143.51 58.42 0)
-      (effects (font (size 1.27 1.27)) hide)
-    )
-    (property "Value" "Earth" (id 1) (at 143.51 55.88 0)
-      (effects (font (size 1.27 1.27)) hide)
-    )
-    (property "Footprint" "" (id 2) (at 143.51 52.07 0)
-      (effects (font (size 1.27 1.27)) hide)
-    )
-    (property "Datasheet" "~" (id 3) (at 143.51 52.07 0)
+  (symbol (lib_id "power:GND") (at 184.15 64.77 90) (unit 1)
+    (in_bom yes) (on_board yes)
+    (property "Reference" "#PWR0106" (id 0) (at 190.5 64.77 0)
+      (effects (font (size 1.27 1.27)) hide)
+    )
+    (property "Value" "GND" (id 1) (at 190.5 64.77 90)
+      (effects (font (size 1.27 1.27)) (justify left))
+    )
+    (property "Footprint" "" (id 2) (at 184.15 64.77 0)
+      (effects (font (size 1.27 1.27)) hide)
+    )
+    (property "Datasheet" "" (id 3) (at 184.15 64.77 0)
       (effects (font (size 1.27 1.27)) hide)
     )
@@
     (pin "7")
   )
-  (symbol (lib_id "power:Earth") (at 130.81 36.83 0) (unit 1)
-    (in_bom yes) (on_board yes) (fields_autoplaced)
-    (property "Reference" "#PWR0101" (id 0) (at 130.81 43.18 0)
-      (effects (font (size 1.27 1.27)) hide)
-    )
-    (property "Value" "Earth" (id 1) (at 130.81 40.64 0)
-      (effects (font (size 1.27 1.27)) hide)
-    )
-    (property "Footprint" "" (id 2) (at 130.81 36.83 0)
-      (effects (font (size 1.27 1.27)) hide)
-    )
-    (property "Datasheet" "~" (id 3) (at 130.81 36.83 0)
+  (symbol (lib_id "power:GND") (at 184.15 77.47 90) (unit 1)
+    (in_bom yes) (on_board yes)
+    (property "Reference" "#PWR0105" (id 0) (at 190.5 77.47 0)
+      (effects (font (size 1.27 1.27)) hide)
+    )
+    (property "Value" "GND" (id 1) (at 190.5 77.47 90)
+      (effects (font (size 1.27 1.27)) (justify left))
+    )
+    (property "Footprint" "" (id 2) (at 184.15 77.47 0)
+      (effects (font (size 1.27 1.27)) hide)
+    )
+    (property "Datasheet" "" (id 3) (at 184.15 77.47 0)
+      (effects (font (size 1.27 1.27)) hide)
+    )
+    (pin "1")
+  )
+  (symbol (lib_id "power:GND") (at 148.59 77.47 270) (unit 1)
+    (in_bom yes) (on_board yes)
+    (property "Reference" "#PWR0108" (id 0) (at 142.24 77.47 0)
+      (effects (font (size 1.27 1.27)) hide)
+    )
+    (property "Value" "GND" (id 1) (at 142.24 77.47 90)
+      (effects (font (size 1.27 1.27)) (justify left))
+    )
+    (property "Footprint" "" (id 2) (at 148.59 77.47 0)
+      (effects (font (size 1.27 1.27)) hide)
+    )
+    (property "Datasheet" "" (id 3) (at 148.59 77.47 0)
+      (effects (font (size 1.27 1.27)) hide)
+    )
+    (pin "1")
+  )
+  (symbol (lib_id "power:GND") (at 130.81 35.56 90) (unit 1)
+    (in_bom yes) (on_board yes) (fields_autoplaced)
+    (property "Reference" "#PWR0102" (id 0) (at 137.16 35.56 0)
+      (effects (font (size 1.27 1.27)) hide)
+    )
+    (property "Value" "GND" (id 1) (at 134.62 35.5599 90)
+      (effects (font (size 1.27 1.27)) (justify right))
+    )
+    (property "Footprint" "" (id 2) (at 130.81 35.56 0)
+      (effects (font (size 1.27 1.27)) hide)
+    )
+    (property "Datasheet" "" (id 3) (at 130.81 35.56 0)
       (effects (font (size 1.27 1.27)) hide)
     )
@@
     (pin "9")
   )
-  (symbol (lib_id "power:Earth") (at 166.37 102.87 180) (unit 1)
-    (in_bom yes) (on_board yes) (fields_autoplaced)
-    (property "Reference" "#PWR?" (id 0) (at 166.37 96.52 0)
-      (effects (font (size 1.27 1.27)) hide)
-    )
-    (property "Value" "Earth" (id 1) (at 166.37 99.06 0)
-      (effects (font (size 1.27 1.27)) hide)
-    )
-    (property "Footprint" "" (id 2) (at 166.37 102.87 0)
-      (effects (font (size 1.27 1.27)) hide)
-    )
-    (property "Datasheet" "~" (id 3) (at 166.37 102.87 0)
+  (symbol (lib_id "power:GND") (at 143.51 52.07 270) (unit 1)
+    (in_bom yes) (on_board yes) (fields_autoplaced)
+    (property "Reference" "#PWR0104" (id 0) (at 137.16 52.07 0)
+      (effects (font (size 1.27 1.27)) hide)
+    )
+    (property "Value" "GND" (id 1) (at 144.78 52.0699 90)
+      (effects (font (size 1.27 1.27)) (justify left))
+    )
+    (property "Footprint" "" (id 2) (at 143.51 52.07 0)
+      (effects (font (size 1.27 1.27)) hide)
+    )
+    (property "Datasheet" "" (id 3) (at 143.51 52.07 0)
       (effects (font (size 1.27 1.27)) hide)
     )
@@
     (pin "3")
   )
+  (symbol (lib_id "power:GND") (at 102.87 66.04 270) (unit 1)
+    (in_bom yes) (on_board yes) (fields_autoplaced)
+    (property "Reference" "#PWR0101" (id 0) (at 96.52 66.04 0)
+      (effects (font (size 1.27 1.27)) hide)
+    )
+    (property "Value" "GND" (id 1) (at 99.06 66.0399 90)
+      (effects (font (size 1.27 1.27)) (justify right))
+    )
+    (property "Footprint" "" (id 2) (at 102.87 66.04 0)
+      (effects (font (size 1.27 1.27)) hide)
+    )
+    (property "Datasheet" "" (id 3) (at 102.87 66.04 0)
+      (effects (font (size 1.27 1.27)) hide)
+    )
+    (pin "1")
+  )
   (sheet_instances
     (path "/" (page "1"))
   )
   (symbol_instances
-    (path "/21d6bcf9-360f-480a-a98d-8ab260d764ed"
-      (reference "#PWR01") (unit 1) (value "Earth") (footprint "")
-    )
-    (path "/4848bfef-8d8f-406b-a025-f4f77ca61ae7"
-      (reference "#PWR02") (unit 1) (value "Earth") (footprint "")
-    )
-    (path "/6eaf7757-5114-4ceb-bc89-5da22eb3e84a"
-      (reference "#PWR0101") (unit 1) (value "Earth") (footprint "")
-    )
-    (path "/a0a28fa4-b96b-4a66-a268-94b1e9e96d9a"
-      (reference "#PWR?") (unit 1) (value "Earth") (footprint "")
+    (path "/e32f3f50-b343-40d8-99dc-2780abeae4b4"
+      (reference "#PWR0101") (unit 1) (value "GND") (footprint "")
+    )
+    (path "/7e35f567-799f-4a55-a604-badd9b6ff54f"
+      (reference "#PWR0102") (unit 1) (value "GND") (footprint "")
+    )
+    (path "/0c392214-7775-4c5e-adad-5b250bff383d"
+      (reference "#PWR0103") (unit 1) (value "GND") (footprint "")
+    )
+    (path "/ae6a83ae-641e-4d3e-bc1b-e98dbf95c78e"
+      (reference "#PWR0104") (unit 1) (value "GND") (footprint "")
+    )
+    (path "/66ba4691-dc56-4cbc-9197-53eafbd24e97"
+      (reference "#PWR0105") (unit 1) (value "GND") (footprint "")
+    )
+    (path "/4c90c559-365f-4931-99b3-b6e0725b5b27"
+      (reference "#PWR0106") (unit 1) (value "GND") (footprint "")
+    )
+    (path "/24767f1c-69a2-47da-8604-20d093b22500"
+      (reference "#PWR0107") (unit 1) (value "GND") (footprint "")
+    )
+    (path "/71b965b3-fb76-48f0-acd7-6c512296c32f"
+      (reference "#PWR0108") (unit 1) (value "GND") (footprint "")
     )
     (path "/9b902966-ba16-4535-a541-f240bc694ecc"

Commit message: board sent out
Changed lines of the file:
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@@
   )
   (symbol (lib_id "Jumper:Jumper_2_Open") (at 212.09 44.45 0) (unit 1)
-    (in_bom yes) (on_board yes) (fields_autoplaced)
-    (property "Reference" "JP2" (id 0) (at 212.09 38.1 0))
+    (in_bom yes) (on_board yes)
+    (property "Reference" "JP2" (id 0) (at 212.09 49.53 0))
     (property "Value" "Jumper_2_Open" (id 1) (at 212.09 40.64 0))
     (property "Footprint" "Connector_PinHeader_2.54mm:PinHeader_1x02_P2.54mm_Vertical" (id 2) (at 212.09 44.45 0)

Commit message: pushed fix for the connector so it a staight through cable
Parts:
- added J5: Conn_01x03_Male, Connector_PinSocket_2.54mm:PinSocket_1x03_P2.54mm_Vertical, symbol Connector:Conn_01x03_Male
Connections:
- net GND: now also J1.8 (Pin_8), J5.2 (Pin_2); no longer J1.3 (Pin_3)
- net SCL_0: now also J1.10 (Pin_10); no longer J1.1 (Pin_1)
- net SCL_1: now also J1.3 (Pin_3); no longer J1.8 (Pin_8)
- net SDA_0: now also J1.1 (Pin_1); no longer J1.10 (Pin_10)
- net SDA_1: now also J1.4 (Pin_4); no longer J1.7 (Pin_7)
- net SWDCLK: now also J1.7 (Pin_7), J5.3 (Pin_3); no longer J1.4 (Pin_4)
- net SWDIO: now also J1.9 (Pin_9), J5.1 (Pin_1); no longer J1.2 (Pin_2)
- net SWO: now also J1.5 (Pin_5); no longer J1.6 (Pin_6)
- net UartTX: now also J1.6 (Pin_6); no longer J1.5 (Pin_5)
- net power_output: now also J1.2 (Pin_2); no longer J1.9 (Pin_9)
Changed lines of the file:
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@@
 (kicad_sch (version 20211123) (generator eeschema)
   (paper "A4")
-  (junction (at 130.81 73.66) (diameter 0) (color 0 0 0 0)
-  )
-  (junction (at 104.14 63.5) (diameter 0) (color 0 0 0 0)
-  )
-  (wire (pts (xy 104.14 63.5) (xy 113.03 63.5))
-    (stroke (width 0) (type default) (color 0 0 0 0))
-  )
-  (wire (pts (xy 102.87 66.04) (xy 113.03 66.04))
+  (junction (at 106.68 63.5) (diameter 0) (color 0 0 0 0)
+  )
+  (junction (at 134.62 73.66) (diameter 0) (color 0 0 0 0)
+  )
+  (wire (pts (xy 101.6 63.5) (xy 106.68 63.5))
+    (stroke (width 0) (type default) (color 0 0 0 0))
+  )
+  (wire (pts (xy 106.68 63.5) (xy 106.68 59.69))
+    (stroke (width 0) (type default) (color 0 0 0 0))
+  )
+  (wire (pts (xy 134.62 78.74) (xy 134.62 73.66))
     (stroke (width 0) (type default) (color 0 0 0 0))
   )
@@
     (stroke (width 0) (type default) (color 0 0 0 0))
   )
-  (wire (pts (xy 99.06 63.5) (xy 104.14 63.5))
-    (stroke (width 0) (type default) (color 0 0 0 0))
-  )
-  (wire (pts (xy 130.81 73.66) (xy 125.73 73.66))
+  (wire (pts (xy 113.03 63.5) (xy 106.68 63.5))
     (stroke (width 0) (type default) (color 0 0 0 0))
   )
@@
     (stroke (width 0) (type default) (color 0 0 0 0))
   )
-  (wire (pts (xy 104.14 59.69) (xy 104.14 63.5))
-    (stroke (width 0) (type default) (color 0 0 0 0))
-  )
   (wire (pts (xy 184.15 44.45) (xy 207.01 44.45))
     (stroke (width 0) (type default) (color 0 0 0 0))
   )
-  (wire (pts (xy 130.81 73.66) (xy 130.81 76.2))
-    (stroke (width 0) (type default) (color 0 0 0 0))
-  )
   (wire (pts (xy 130.81 35.56) (xy 121.92 35.56))
     (stroke (width 0) (type default) (color 0 0 0 0))
@@
     (stroke (width 0) (type default) (color 0 0 0 0))
   )
-  (wire (pts (xy 135.89 73.66) (xy 130.81 73.66))
-    (stroke (width 0) (type default) (color 0 0 0 0))
+  (wire (pts (xy 134.62 73.66) (xy 125.73 73.66))
+    (stroke (width 0) (type default) (color 0 0 0 0))
+  )
+  (wire (pts (xy 139.7 73.66) (xy 134.62 73.66))
+    (stroke (width 0) (type default) (color 0 0 0 0))
+  )
+  (label "SCL_1" (at 113.03 66.04 180)
+    (effects (font (size 1.27 1.27)) (justify right bottom))
   )
   (label "SWDCLK" (at 121.92 33.02 0)
@@
     (effects (font (size 1.27 1.27)) (justify right bottom))
   )
+  (label "SWDCLK" (at 203.2 96.52 0)
+    (effects (font (size 1.27 1.27)) (justify left bottom))
+  )
   (label "TRST" (at 148.59 46.99 180)
     (effects (font (size 1.27 1.27)) (justify right bottom))
@@
     (effects (font (size 1.27 1.27)) (justify left bottom))
   )
-  (label "power_output" (at 113.03 73.66 180)
-    (effects (font (size 1.27 1.27)) (justify right bottom))
-  )
-  (label "SCL_0" (at 104.14 59.69 90)
-    (effects (font (size 1.27 1.27)) (justify left bottom))
-  )
-  (label "SWDCLK" (at 125.73 66.04 0)
+  (label "power_output" (at 125.73 63.5 0)
+    (effects (font (size 1.27 1.27)) (justify left bottom))
+  )
+  (label "SDA_0" (at 106.68 59.69 90)
     (effects (font (size 1.27 1.27)) (justify left bottom))
   )
@@
     (effects (font (size 1.27 1.27)) (justify right bottom))
   )
+  (label "SWDIO" (at 113.03 73.66 180)
+    (effects (font (size 1.27 1.27)) (justify right bottom))
+  )
   (label "SWO" (at 148.59 49.53 180)
     (effects (font (size 1.27 1.27)) (justify right bottom))
   )
+  (label "UartTX" (at 125.73 68.58 0)
+    (effects (font (size 1.27 1.27)) (justify left bottom))
+  )
   (label "SDA_0" (at 118.11 104.14 180)
     (effects (font (size 1.27 1.27)) (justify right bottom))
@@
     (effects (font (size 1.27 1.27)) (justify left bottom))
   )
-  (label "SCL_1" (at 125.73 71.12 0)
+  (label "SWDIO" (at 203.2 91.44 0)
     (effects (font (size 1.27 1.27)) (justify left bottom))
   )
@@
     (effects (font (size 1.27 1.27)) (justify right bottom))
   )
+  (label "SWDCLK" (at 113.03 71.12 180)
+    (effects (font (size 1.27 1.27)) (justify right bottom))
+  )
   (label "VTREF" (at 184.15 49.53 0)
     (effects (font (size 1.27 1.27)) (justify left bottom))
@@
     (effects (font (size 1.27 1.27)) (justify left bottom))
   )
-  (label "TRST" (at 135.89 73.66 0)
+  (label "SDA_1" (at 125.73 66.04 0)
     (effects (font (size 1.27 1.27)) (justify left bottom))
   )
@@
     (effects (font (size 1.27 1.27)) (justify left bottom))
   )
-  (label "SDA_1" (at 113.03 71.12 180)
-    (effects (font (size 1.27 1.27)) (justify right bottom))
-  )
   (label "SCL_1" (at 130.81 106.68 0)
     (effects (font (size 1.27 1.27)) (justify left bottom))
   )
-  (label "SWDIO" (at 125.73 63.5 0)
-    (effects (font (size 1.27 1.27)) (justify left bottom))
-  )
   (label "SWDCLK" (at 148.59 41.91 180)
     (effects (font (size 1.27 1.27)) (justify right bottom))
@@
     (effects (font (size 1.27 1.27)) (justify left bottom))
   )
-  (label "UartTX" (at 111.76 68.58 180)
-    (effects (font (size 1.27 1.27)) (justify right bottom))
-  )
-  (label "SWO" (at 125.73 68.58 0)
-    (effects (font (size 1.27 1.27)) (justify left bottom))
-  )
-  (label "VTREF" (at 99.06 63.5 180)
+  (label "SWO" (at 111.76 68.58 180)
+    (effects (font (size 1.27 1.27)) (justify right bottom))
+  )
+  (label "SCL_0" (at 134.62 78.74 270)
     (effects (font (size 1.27 1.27)) (justify right bottom))
   )
@@
     (effects (font (size 1.27 1.27)) (justify left bottom))
   )
-  (label "SDA_0" (at 130.81 76.2 270)
+  (label "TRST" (at 101.6 63.5 180)
     (effects (font (size 1.27 1.27)) (justify right bottom))
   )
   (label "SWO" (at 130.81 101.6 0)
+    (effects (font (size 1.27 1.27)) (justify left bottom))
+  )
+  (label "VTREF" (at 139.7 73.66 0)
     (effects (font (size 1.27 1.27)) (justify left bottom))
   )
@@
     (pin "2")
   )
+  (symbol (lib_id "Connector:Conn_01x03_Male") (at 198.12 93.98 0) (unit 1)
+    (in_bom yes) (on_board yes) (fields_autoplaced)
+    (property "Reference" "J5" (id 0) (at 198.755 86.36 0))
+    (property "Value" "Conn_01x03_Male" (id 1) (at 198.755 88.9 0))
+    (property "Footprint" "Connector_PinSocket_2.54mm:PinSocket_1x03_P2.54mm_Vertical" (id 2) (at 198.12 93.98 0)
+      (effects (font (size 1.27 1.27)) hide)
+    )
+    (property "Datasheet" "~" (id 3) (at 198.12 93.98 0)
+      (effects (font (size 1.27 1.27)) hide)
+    )
+    (pin "1")
+    (pin "2")
+    (pin "3")
+  )
   (symbol (lib_id "power:GND") (at 184.15 64.77 90) (unit 1)
     (in_bom yes) (on_board yes)
@@
     )
     (property "Datasheet" "" (id 3) (at 184.15 64.77 0)
+      (effects (font (size 1.27 1.27)) hide)
+    )
+    (pin "1")
+  )
+  (symbol (lib_id "power:GND") (at 125.73 71.12 90) (unit 1)
+    (in_bom yes) (on_board yes) (fields_autoplaced)
+    (property "Reference" "#PWR?" (id 0) (at 132.08 71.12 0)
+      (effects (font (size 1.27 1.27)) hide)
+    )
+    (property "Value" "GND" (id 1) (at 129.54 71.1199 90)
+      (effects (font (size 1.27 1.27)) (justify right))
+    )
+    (property "Footprint" "" (id 2) (at 125.73 71.12 0)
+      (effects (font (size 1.27 1.27)) hide)
+    )
+    (property "Datasheet" "" (id 3) (at 125.73 71.12 0)
       (effects (font (size 1.27 1.27)) hide)
     )
@@
     (pin "3")
   )
-  (symbol (lib_id "power:GND") (at 102.87 66.04 270) (unit 1)
-    (in_bom yes) (on_board yes) (fields_autoplaced)
-    (property "Reference" "#PWR0101" (id 0) (at 96.52 66.04 0)
-      (effects (font (size 1.27 1.27)) hide)
-    )
-    (property "Value" "GND" (id 1) (at 99.06 66.0399 90)
+  (symbol (lib_id "power:GND") (at 203.2 93.98 90) (unit 1)
+    (in_bom yes) (on_board yes)
+    (property "Reference" "#PWR0109" (id 0) (at 209.55 93.98 0)
+      (effects (font (size 1.27 1.27)) hide)
+    )
+    (property "Value" "GND" (id 1) (at 207.01 93.9801 90)
       (effects (font (size 1.27 1.27)) (justify right))
     )
-    (property "Footprint" "" (id 2) (at 102.87 66.04 0)
-      (effects (font (size 1.27 1.27)) hide)
-    )
-    (property "Datasheet" "" (id 3) (at 102.87 66.04 0)
+    (property "Footprint" "" (id 2) (at 203.2 93.98 0)
+      (effects (font (size 1.27 1.27)) hide)
+    )
+    (property "Datasheet" "" (id 3) (at 203.2 93.98 0)
       (effects (font (size 1.27 1.27)) hide)
     )
@@
   )
   (symbol_instances
-    (path "/e32f3f50-b343-40d8-99dc-2780abeae4b4"
-      (reference "#PWR0101") (unit 1) (value "GND") (footprint "")
-    )
     (path "/7e35f567-799f-4a55-a604-badd9b6ff54f"
       (reference "#PWR0102") (unit 1) (value "GND") (footprint "")
@@
       (reference "#PWR0108") (unit 1) (value "GND") (footprint "")
     )
+    (path "/f6bbcec5-47eb-4924-a608-c6c5ca5e14ea"
+      (reference "#PWR0109") (unit 1) (value "GND") (footprint "")
+    )
+    (path "/4dd09e6e-777d-40bd-be58-fc9ee457c32d"
+      (reference "#PWR?") (unit 1) (value "GND") (footprint "")
+    )
     (path "/9b902966-ba16-4535-a541-f240bc694ecc"
       (reference "J1") (unit 1) (value "Conn_02x05_Odd_Even") (footprint "LocalFootprints:3220-10-0300-00-TR")
@@
       (reference "J4") (unit 1) (value "BM03B-SRSS-TBLFSN") (footprint "JST:BM03B-SRSS-TBLFSN")
     )
+    (path "/336d36fa-a7d0-4e31-b97e-7e2f57518017"
+      (reference "J5") (unit 1) (value "Conn_01x03_Male") (footprint "Connector_PinSocket_2.54mm:PinSocket_1x03_P2.54mm_Vertical")
+    )
     (path "/0477c905-d10c-47a4-9a1e-4219e82ce5fc"
